Commit message: Got rid of dup pi

File: robotiq_85_description/urdf/robotiq_85_gripper.urdf.xacro (robot description, xacro)
@@ -2,5 +2,4 @@
 <robot name="robotiq_85_gripper" xmlns:xacro="http://ros.org/wiki/xacro">
     <xacro:include filename="$(find robotiq_85_description)/urdf/robotiq_85_gripper.transmission.xacro" />
-    <xacro:property name="pi" value="3.14159"/>
     <xacro:macro name="robotiq_85_gripper" params="prefix parent *origin">
         <joint name="${prefix}robotiq_85_base_joint" type="fixed">
